Commit message: Updated URDF and added ros2_control

File: description/lidar.xacro (robot description, xacro)
@@ -2,7 +2,7 @@
 <robot xmlns:xacro="http://www.ros.org/wiki/xacro">
    <joint name="laser_joint" type="fixed">
-      <parent link="base_link"/>
+      <parent link="chassis"/>
       <child link="laser_frame"/>
-      <origin xyz="0.0 0.0 0.5975"/>
+      <origin xyz="${chassis_length/2} 0 ${chassis_height + head_height + (wheel_thickness/2)}"/>
    </joint>
    <link name="laser_frame">
@@ -18,5 +18,5 @@
          </geometry>
       </collision>
-       <xacro:inertial_cylinder mass="0.15" length="0.035" radius="0.04">
+       <xacro:inertial_cylinder mass="0.170" length="0.035" radius="0.04">
          <origin xyz="0.0 0.0 0.0" rpy="0.0 0.0 0.0"/>
       </xacro:inertial_cylinder>
@@ -26,5 +26,5 @@
       <sensor name="laser" type="ray">
          <pose>0 0 0 0 0 0</pose>
-         <visualize>true</visualize>
+         <visualize>false</visualize>
          <update_rate>10</update_rate>
          <ray>
@@ -43,5 +43,5 @@
          <plugin name="laser_controller" filename="libgazebo_ros_ray_sensor.so">
             <ros>
-               <argument>~/out:=scan</argument>
+               <remapping>~/out:=scan</remapping>
             </ros>
             <output_type>sensor_msgs/LaserScan</output_type>

File: description/robot.urdf.xacro (robot description, xacro)
@@ -1,6 +1,20 @@
 <?xml version="1.0" encoding="UTF-8"?>
 <robot xmlns:xacro="http://wiki.ros.org/wiki/xacro" name="robot">
+   <!-- args -->
+   <xacro:arg name="use_ros2_control" default="true"/>
+   <!-- initialize xacro properties -->
+   <xacro:include filename="inertial_macros.xacro"/>
+   <xacro:include filename="properties.xacro"/>
+   <!-- initialize robot URDF -->
    <xacro:include filename="robot_core.xacro"/>
-   <xacro:include filename="gazebo_control.xacro"/>
+   <!-- initialize ros2_control -->
+   <xacro:if value="$(arg use_ros2_control)">
+      <xacro:include filename="ros2_control.xacro"/>
+   </xacro:if>
+   <xacro:unless value="$(arg use_ros2_control)">
+      <xacro:include filename="gazebo_control.xacro"/>
+   </xacro:unless>
+   <!-- initialize sensors -->
    <xacro:include filename="lidar.xacro"/>
+   <xacro:include filename="camera.xacro"/>
 </robot>

File: description/robot_core.xacro (robot description, xacro)
@@ -1,40 +1,4 @@
 <?xml version="1.0" encoding="UTF-8"?>
 <robot xmlns:xacro="http://wiki.ros.org/wiki/xacro">
-   <xacro:include filename="inertial_macros.xacro"/>
-   <xacro:property name="chassis_length" value="0.170"/>
-   <xacro:property name="chassis_width" value="0.275"/>
-   <xacro:property name="chassis_height" value="0.36"/>
-   <xacro:property name="chassis_mass" value="2.5"/>
-   <xacro:property name="head_length" value="0.230"/>
-   <xacro:property name="head_width" value="0.385"/>
-   <xacro:property name="head_height" value="0.220"/>
-   <xacro:property name="head_mass" value="0.7"/>
-   <xacro:property name="front_caster_holder_length" value="0.160"/>
-   <xacro:property name="front_caster_holder_width" value="0.085"/>
-   <xacro:property name="front_caster_holder_height" value="0.050"/>
-   <xacro:property name="front_caster_holder_mass" value="0.08"/>
-   <xacro:property name="back_wheel_holder_length" value="0.05"/>
-   <xacro:property name="back_wheel_holder_width" value="0.1"/>
-   <xacro:property name="back_wheel_holder_height" value="0.02"/>
-   <xacro:property name="back_wheel_holder_mass" value="0.05"/>
-   <xacro:property name="wheel_radius" value="0.04"/>
-   <xacro:property name="wheel_thickness" value="0.035"/>
-   <xacro:property name="wheel_mass" value="0.15"/>
-   <xacro:property name="wheel_offset_x" value="0.11"/>
-   <xacro:property name="wheel_offset_y" value="0.1375"/>
-   <xacro:property name="wheel_offset_z" value="0.030"/>
-   <xacro:property name="caster_wheel_radius" value="0.04"/>
-   <xacro:property name="caster_wheel_mass" value="0.1"/>
-   <xacro:property name="caster_wheel_offset_x" value="0.120"/>
-   <xacro:property name="caster_wheel_offset_z" value="${wheel_offset_z - wheel_radius + caster_wheel_radius}"/>
-   <material name="white">
-      <color rgba="1 1 1 1"/>
-   </material>
-   <material name="black">
-      <color rgba="0 0 0 1"/>
-   </material>
-   <material name="grey" >
-        <color rgba="0.5725490196078431 0.5843137254901961 0.5686274509803921 1.0" />
-    </material>
    <!-- BASE LINK -->
    <link name="base_link"></link>
@@ -54,5 +18,5 @@
       </visual>
       <collision>
-         <origin xyz="0.085 0.0 0.18"/>
+         <origin xyz="${chassis_length/2} 0.0 ${chassis_height/2}"/>
          <geometry>
             <box size="${chassis_length} ${chassis_width} ${chassis_height}"/>
@@ -67,6 +31,6 @@
    </gazebo>
    <joint name="head_joint" type="fixed">
-      <origin xyz="0.0 0.0 ${chassis_height + (head_height/2)}"/>
-      <parent link="base_link"/>
+      <origin xyz="${chassis_length/2} 0.0 ${chassis_height + (head_height/2)}"/>
+      <parent link="chassis"/>
       <child link="head"/>
    </joint>
@@ -125,12 +89,12 @@
    <link name="left_back_caster_holder">
       <visual>
-         <origin xyz="-${back_wheel_holder_length/2} -${back_wheel_holder_width/2} ${back_wheel_holder_height/2}"/>
-         <geometry>
-            <box size="${back_wheel_holder_length} ${back_wheel_holder_width} ${back_wheel_holder_height}"/>
-         </geometry>
-         <material name="white"/>
-      </visual>
-      <collision>
-         <origin xyz="-${back_wheel_holder_length/2} -${back_wheel_holder_width/2} ${back_wheel_holder_height/2}"/>
+         <origin xyz="-${back_wheel_holder_length/2} -${back_wheel_holder_width/2} -${back_wheel_holder_height/2}"/>
+         <geometry>
+            <box size="${back_wheel_holder_length} ${back_wheel_holder_width} ${back_wheel_holder_height}"/>
+         </geometry>
+         <material name="white"/>
+      </visual>
+      <collision>
+         <origin xyz="-${back_wheel_holder_length/2} -${back_wheel_holder_width/2} -${back_wheel_holder_height/2}"/>
          <geometry>
             <box size="${back_wheel_holder_length} ${back_wheel_holder_width} ${back_wheel_holder_height}"/>
@@ -151,12 +115,12 @@
    <link name="right_back_caster_holder">
       <visual>
-         <origin xyz="-${back_wheel_holder_length/2} ${back_wheel_holder_width/2} ${back_wheel_holder_height/2}"/>
-         <geometry>
-            <box size="${back_wheel_holder_length} ${back_wheel_holder_width} ${back_wheel_holder_height}"/>
-         </geometry>
-         <material name="white"/>
-      </visual>
-      <collision>
-         <origin xyz="-${back_wheel_holder_length/2} ${back_wheel_holder_width/2} ${back_wheel_holder_height/2}"/>
+         <origin xyz="-${back_wheel_holder_length/2} ${back_wheel_holder_width/2} -${back_wheel_holder_height/2}"/>
+         <geometry>
+            <box size="${back_wheel_holder_length} ${back_wheel_holder_width} ${back_wheel_holder_height}"/>
+         </geometry>
+         <material name="white"/>
+      </visual>
+      <collision>
+         <origin xyz="-${back_wheel_holder_length/2} ${back_wheel_holder_width/2} -${back_wheel_holder_height/2}"/>
          <geometry>
             <box size="${back_wheel_holder_length} ${back_wheel_holder_width} ${back_wheel_holder_height}"/>
@@ -186,6 +150,7 @@
       <collision>
          <geometry>
-            <cylinder radius="${wheel_radius}" length="${wheel_thickness}"/>
-         </geometry>
+            <sphere radius="${wheel_radius}"/>
+         </geometry>
+         <material name="orange"/>
       </collision>
       <xacro:inertial_cylinder mass="${wheel_mass}" length="${wheel_thickness}" radius="${wheel_radius}">
@@ -211,6 +176,7 @@
       <collision>
          <geometry>
-            <cylinder radius="${wheel_radius}" length="${wheel_thickness}"/>
-         </geometry>
+            <sphere radius="${wheel_radius}"/>
+         </geometry>
+         <material name="bloodorange"/>
       </collision>
        <xacro:inertial_cylinder mass="${wheel_mass}" length="${wheel_thickness}" radius="${wheel_radius}">

Commit message: switching rpi

File: description/lidar.xacro (robot description, xacro)
@@ -2,7 +2,7 @@
 <robot xmlns:xacro="http://www.ros.org/wiki/xacro">
    <joint name="laser_joint" type="fixed">
-      <parent link="chassis"/>
+      <parent link="base_link"/>
       <child link="laser_frame"/>
-      <origin xyz="${chassis_length/2} 0 ${chassis_height + head_height + (wheel_thickness/2)}"/>
+      <origin xyz="0 0 ${chassis_height + head_height + (wheel_thickness/2)}"/>
    </joint>
    <link name="laser_frame">

File: description/ros2_control.xacro (robot description, xacro)
@@ -1,5 +1,33 @@
 <?xml version="1.0" encoding="UTF-8"?>
 <robot xmlns:xacro="http://www.ros.org/wiki/xacro">
-   <ros2_control name="GazeboSystem" type="system">
+   <ros2_control name="RealRobot" type="system">
+      <hardware>
+         <plugin>diffdrive_arduino/DiffDriveArduino</plugin>
+         <param name="left_wheel_name">left_wheel_joint</param>
+         <param name="right_wheel_name">right_wheel_joint</param>
+         <param name="loop_rate">30</param>
+         <param name="device">/dev/ttyACM0</param>
+         <param name="baud_rate">57600</param>
+         <param name="timeout">1000</param>
+         <param name="enc_counts_per_rev">2800</param>
+      </hardware>
+      <joint name="left_wheel_joint">
+         <command_interface name="velocity">
+            <param name="min">-10</param>
+            <param name="max">10</param>
+         </command_interface>
+         <state_interface name="velocity"/>
+         <state_interface name="position"/>
+      </joint>
+      <joint name="right_wheel_joint">
+         <command_interface name="velocity">
+            <param name="min">-10</param>
+            <param name="max">10</param>
+         </command_interface>
+         <state_interface name="velocity"/>
+         <state_interface name="position"/>
+      </joint>
+   </ros2_control>
+   <!-- <ros2_control name="GazeboSystem" type="system">
       <hardware>
          <plugin>gazebo_ros2_control/GazeboSystem</plugin>
@@ -21,5 +49,5 @@
          <state_interface name="position"/>
       </joint>
-   </ros2_control>
+   </ros2_control> -->
    <gazebo>
       <plugin name="gazebo_ros2_control" filename="libgazebo_ros2_control.so">

Commit message: added ros2_control

File: description/lidar.xacro (robot description, xacro)
@@ -2,7 +2,7 @@
 <robot xmlns:xacro="http://www.ros.org/wiki/xacro">
    <joint name="laser_joint" type="fixed">
-      <parent link="base_link"/>
+      <parent link="chassis"/>
       <child link="laser_frame"/>
-      <origin xyz="0 0 ${chassis_height + head_height + (wheel_thickness/2)}"/>
+      <origin xyz="${chassis_length/2} 0 ${chassis_height + head_height + (wheel_thickness/2)}"/>
    </joint>
    <link name="laser_frame">

File: description/ros2_control.xacro (robot description, xacro)
@@ -10,5 +10,5 @@
          <param name="baud_rate">57600</param>
          <param name="timeout">1000</param>
-         <param name="enc_counts_per_rev">2800</param>
+         <param name="enc_counts_per_rev">2803</param>
       </hardware>
       <joint name="left_wheel_joint">
