Commit message: Updated robot URDF

File: description/robot.urdf.xacro (robot description, xacro)
@@ -2,3 +2,5 @@
 <robot xmlns:xacro="http://wiki.ros.org/wiki/xacro" name="robot">
    <xacro:include filename="robot_core.xacro"/>
+   <xacro:include filename="gazebo_control.xacro"/>
+   <xacro:include filename="lidar.xacro"/>
 </robot>

File: description/robot_core.xacro (robot description, xacro)
@@ -2,4 +2,30 @@
 <robot xmlns:xacro="http://wiki.ros.org/wiki/xacro">
    <xacro:include filename="inertial_macros.xacro"/>
+   <xacro:property name="chassis_length" value="0.170"/>
+   <xacro:property name="chassis_width" value="0.275"/>
+   <xacro:property name="chassis_height" value="0.36"/>
+   <xacro:property name="chassis_mass" value="2.5"/>
+   <xacro:property name="head_length" value="0.230"/>
+   <xacro:property name="head_width" value="0.385"/>
+   <xacro:property name="head_height" value="0.220"/>
+   <xacro:property name="head_mass" value="0.7"/>
+   <xacro:property name="front_caster_holder_length" value="0.160"/>
+   <xacro:property name="front_caster_holder_width" value="0.085"/>
+   <xacro:property name="front_caster_holder_height" value="0.050"/>
+   <xacro:property name="front_caster_holder_mass" value="0.08"/>
+   <xacro:property name="back_wheel_holder_length" value="0.05"/>
+   <xacro:property name="back_wheel_holder_width" value="0.1"/>
+   <xacro:property name="back_wheel_holder_height" value="0.02"/>
+   <xacro:property name="back_wheel_holder_mass" value="0.05"/>
+   <xacro:property name="wheel_radius" value="0.04"/>
+   <xacro:property name="wheel_thickness" value="0.035"/>
+   <xacro:property name="wheel_mass" value="0.15"/>
+   <xacro:property name="wheel_offset_x" value="0.11"/>
+   <xacro:property name="wheel_offset_y" value="0.1375"/>
+   <xacro:property name="wheel_offset_z" value="0.030"/>
+   <xacro:property name="caster_wheel_radius" value="0.04"/>
+   <xacro:property name="caster_wheel_mass" value="0.1"/>
+   <xacro:property name="caster_wheel_offset_x" value="0.120"/>
+   <xacro:property name="caster_wheel_offset_z" value="${wheel_offset_z - wheel_radius + caster_wheel_radius}"/>
    <material name="white">
       <color rgba="1 1 1 1"/>
@@ -8,12 +34,12 @@
       <color rgba="0 0 0 1"/>
    </material>
-   <material name="gray">
-      <color rgba="0.8 0.78 0.78 1"/>
-   </material>
+   <material name="grey" >
+        <color rgba="0.5725490196078431 0.5843137254901961 0.5686274509803921 1.0" />
+    </material>
    <!-- BASE LINK -->
    <link name="base_link"></link>
    <!-- CHASSIS -->
    <joint name="chassis_joint" type="fixed">
-      <origin xyz="-0.0825 0.0 0.0"/>
+      <origin xyz="-${chassis_length/2} 0.0 0.0"/>
       <parent link="base_link"/>
       <child link="chassis"/>
@@ -21,22 +47,51 @@
    <link name="chassis">
       <visual>
-         <origin xyz="0.0825 0.0 0.29"/>
-         <geometry>
-            <box size="0.165 0.319 0.575"/>
-         </geometry>
-         <material name="white"/>
-      </visual>
-      <collision>
-         <origin xyz="0.0825 0.0 0.29"/>
-         <geometry>
-            <box size="0.165 0.319 0.575"/>
-         </geometry>
-      </collision>
-      <xacro:inertial_box mass="2" x="0.165" y="0.319" z="0.575">
-         <origin xyz="0.0825 0.0 0.29" rpy="0.0 0.0 0.0"/>
-      </xacro:inertial_box>
-   </link>
+         <origin xyz="${chassis_length/2} 0.0 ${chassis_height/2}"/>
+         <geometry>
+            <box size="${chassis_length} ${chassis_width} ${chassis_height}"/>
+         </geometry>
+         <material name="white"/>
+      </visual>
+      <collision>
+         <origin xyz="0.085 0.0 0.18"/>
+         <geometry>
+            <box size="${chassis_length} ${chassis_width} ${chassis_height}"/>
+         </geometry>
+      </collision>
+      <xacro:inertial_box mass="2" x="${chassis_length}" y="${chassis_width}" z="${chassis_height}">
+         <origin xyz="${chassis_length} 0.0 ${chassis_height/2}" rpy="0.0 0.0 0.0"/>
+      </xacro:inertial_box>
+   </link>
+   <gazebo reference="chassis">
+      <material>Gazebo/White</material>
+   </gazebo>
+   <joint name="head_joint" type="fixed">
+      <origin xyz="0.0 0.0 ${chassis_height + (head_height/2)}"/>
+      <parent link="base_link"/>
+      <child link="head"/>
+   </joint>
+   <link name="head">
+      <visual>
+         <origin xyz="0.0 0.0 0.0"/>
+         <geometry>
+            <box size="${head_length} ${head_width} ${head_height}"/>
+         </geometry>
+         <material name="white"/>
+      </visual>
+      <collision>
+         <origin xyz="0.0 0.0 0.0"/>
+         <geometry>
+            <box size="${head_length} ${head_width} ${head_height}"/>
+         </geometry>
+      </collision>
+      <xacro:inertial_box mass="2" x="${head_length}" y="${head_width}" z="${head_height}">
+         <origin xyz="0.0 0.0 0.0" rpy="0.0 0.0 0.0"/>
+      </xacro:inertial_box>
+   </link>
+   <gazebo reference="head">
+      <material>Gazebo/White</material>
+   </gazebo>
    <joint name="front_caster_holder_joint" type="fixed">
-      <origin xyz="0.165 0.0 0.0"/>
+      <origin xyz="${chassis_length} 0.0 0.0"/>
       <parent link="chassis"/>
       <child link="front_caster_holder"/>
@@ -44,48 +99,80 @@
    <link name="front_caster_holder">
       <visual>
-         <origin xyz="0.08 0.0 0.025"/>
-         <geometry>
-            <box size="0.160 0.085 0.050"/>
-         </geometry>
-         <material name="white"/>
-      </visual>
-      <collision>
-         <origin xyz="0.08 0.0 0.025"/>
-         <geometry>
-            <box size="0.160 0.085 0.050"/>
-         </geometry>
-      </collision>
-      <xacro:inertial_box mass="0.08" x="0.16" y="0.085" z="0.050">
-         <origin xyz="0.08 0.0 0.025" rpy="0.0 0.0 0.0"/>
-      </xacro:inertial_box>
-   </link>
-   <joint name="back_caster_holder_joint" type="fixed">
-      <origin xyz="0.0 0.0 0.0"/>
+         <origin xyz="${front_caster_holder_length/2} 0.0 ${front_caster_holder_height/2}"/>
+         <geometry>
+            <box size="${front_caster_holder_length} ${front_caster_holder_width} ${front_caster_holder_height}"/>
+         </geometry>
+         <material name="white"/>
+      </visual>
+      <collision>
+         <origin xyz="${front_caster_holder_length/2} 0.0 ${front_caster_holder_height/2}"/>
+         <geometry>
+            <box size="${front_caster_holder_length} ${front_caster_holder_width} ${front_caster_holder_height}"/>
+         </geometry>
+      </collision>
+      <xacro:inertial_box mass="${front_caster_holder_mass}" x="${front_caster_holder_length}" y="${front_caster_holder_width}" z="${front_caster_holder_height}">
+         <origin xyz="${front_caster_holder_length/2} 0.0 ${front_caster_holder_height/2}"/>
+      </xacro:inertial_box>
+   </link>
+   <gazebo reference="front_caster_holder">
+      <material>Gazebo/White</material>
+   </gazebo>
+   <joint name="left_back_wheel_holder_joint" type="fixed">
+      <origin xyz="0.0 ${chassis_width/2} 0.0"/>
       <parent link="chassis"/>
-      <child link="back_caster_holder"/>
-   </joint>
-   <link name="back_caster_holder">
-      <visual>
-         <origin xyz="-0.035 0.0 0.01"/>
-         <geometry>
-            <box size="0.07 0.1 0.02"/>
-         </geometry>
-         <material name="white"/>
-      </visual>
-      <collision>
-         <origin xyz="-0.035 0.0 0.01"/>
-         <geometry>
-            <box size="0.07 0.1 0.02"/>
-         </geometry>
-      </collision>
-      <xacro:inertial_box mass="0.05" x="0.07" y="0.1" z="0.02">
-         <origin xyz="-0.035 0.0 0.01" rpy="0.0 0.0 0.0"/>
-      </xacro:inertial_box>
-   </link>
+      <child link="left_back_caster_holder"/>
+   </joint>
+   <link name="left_back_caster_holder">
+      <visual>
+         <origin xyz="-${back_wheel_holder_length/2} -${back_wheel_holder_width/2} ${back_wheel_holder_height/2}"/>
+         <geometry>
+            <box size="${back_wheel_holder_length} ${back_wheel_holder_width} ${back_wheel_holder_height}"/>
+         </geometry>
+         <material name="white"/>
+      </visual>
+      <collision>
+         <origin xyz="-${back_wheel_holder_length/2} -${back_wheel_holder_width/2} ${back_wheel_holder_height/2}"/>
+         <geometry>
+            <box size="${back_wheel_holder_length} ${back_wheel_holder_width} ${back_wheel_holder_height}"/>
+         </geometry>
+      </collision>
+      <xacro:inertial_box mass="${back_wheel_holder_mass}" x="${back_wheel_holder_length}" y="${back_wheel_holder_width}" z="${back_wheel_holder_height}">
+         <origin xyz="-${back_wheel_holder_length/2} -${back_wheel_holder_width/2} ${back_wheel_holder_height/2}" rpy="0.0 0.0 0.0"/>
+      </xacro:inertial_box>
+   </link>
+   <gazebo reference="left_back_caster_holder">
+      <material>Gazebo/White</material>
+   </gazebo>
+   <joint name="right_back_caster_holder_joint" type="fixed">
+      <origin xyz="0.0 -${chassis_width/2} 0.0"/>
+      <parent link="chassis"/>
+      <child link="right_back_caster_holder"/>
+   </joint>
+   <link name="right_back_caster_holder">
+      <visual>
+         <origin xyz="-${back_wheel_holder_length/2} ${back_wheel_holder_width/2} ${back_wheel_holder_height/2}"/>
+         <geometry>
+            <box size="${back_wheel_holder_length} ${back_wheel_holder_width} ${back_wheel_holder_height}"/>
+         </geometry>
+         <material name="white"/>
+      </visual>
+      <collision>
+         <origin xyz="-${back_wheel_holder_length/2} ${back_wheel_holder_width/2} ${back_wheel_holder_height/2}"/>
+         <geometry>
+            <box size="${back_wheel_holder_length} ${back_wheel_holder_width} ${back_wheel_holder_height}"/>
+         </geometry>
+      </collision>
+      <xacro:inertial_box mass="${back_wheel_holder_mass}" x="${back_wheel_holder_length}" y="${back_wheel_holder_width}" z="${back_wheel_holder_height}">
+         <origin xyz="-${back_wheel_holder_length/2} ${back_wheel_holder_width/2} ${back_wheel_holder_height/2}" rpy="0.0 0.0 0.0"/>
+      </xacro:inertial_box>
+   </link>
+   <gazebo reference="right_back_caster_holder">
+      <material>Gazebo/White</material>
+   </gazebo>
    <!-- WHEELS -->
    <joint name="left_wheel_joint" type="continuous">
       <parent link="base_link"/>
       <child link="left_wheel"/>
-      <origin xyz="0 0.177 -0.025" rpy="-${pi/2} 0 0"/>
+      <origin xyz="-${wheel_offset_x} ${wheel_offset_y} -${wheel_offset_z}" rpy="-${pi/2} 0 0"/>
       <axis xyz="0.0 0.0 1"/>
    </joint>
@@ -93,5 +180,5 @@
       <visual>
          <geometry>
-            <cylinder radius="0.041" length="0.035"/>
+            <cylinder radius="${wheel_radius}" length="${wheel_thickness}"/>
          </geometry>
          <material name="black"/>
@@ -99,15 +186,18 @@
       <collision>
          <geometry>
-            <cylinder radius="0.041" length="0.035"/>
-         </geometry>
-      </collision>
-      <xacro:inertial_cylinder mass="0.15" length="0.035" radius="0.041">
+            <cylinder radius="${wheel_radius}" length="${wheel_thickness}"/>
+         </geometry>
+      </collision>
+      <xacro:inertial_cylinder mass="${wheel_mass}" length="${wheel_thickness}" radius="${wheel_radius}">
          <origin xyz="0.0 0.0 0.0" rpy="0.0 0.0 0.0"/>
       </xacro:inertial_cylinder>
    </link>
+   <gazebo reference="left_wheel">
+      <material>Gazebo/Black</material>
+   </gazebo>
    <joint name="right_wheel_joint" type="continuous">
       <parent link="base_link"/>
       <child link="right_wheel"/>
-      <origin xyz="0 -0.177 -0.025" rpy="${pi/2} 0 0"/>
+      <origin xyz="-${wheel_offset_x} -${wheel_offset_y} -${wheel_offset_z}" rpy="${pi/2} 0 0"/>
       <axis xyz="0.0 0.0 -1"/>
    </joint>
@@ -115,5 +205,5 @@
       <visual>
          <geometry>
-            <cylinder radius="0.041" length="0.035"/>
+            <cylinder radius="${wheel_radius}" length="${wheel_thickness}"/>
          </geometry>
          <material name="black"/>
@@ -121,16 +211,19 @@
       <collision>
          <geometry>
-            <cylinder radius="0.041" length="0.035"/>
-         </geometry>
-      </collision>
-       <xacro:inertial_cylinder mass="0.15" length="0.035" radius="0.041">
+            <cylinder radius="${wheel_radius}" length="${wheel_thickness}"/>
+         </geometry>
+      </collision>
+       <xacro:inertial_cylinder mass="${wheel_mass}" length="${wheel_thickness}" radius="${wheel_radius}">
          <origin xyz="0.0 0.0 0.0" rpy="0.0 0.0 0.0"/>
       </xacro:inertial_cylinder>
    </link>
+   <gazebo reference="right_wheel">
+      <material>Gazebo/Black</material>
+   </gazebo>
    <!-- CASTER WHEELS -->
    <joint name="front_caster_wheel_joint" type="fixed">
       <parent link="front_caster_holder"/>
       <child link="front_caster_wheel"/>
-      <origin xyz="0.120 0.0 -0.025"/>
+      <origin xyz="${caster_wheel_offset_x} 0.0 -${caster_wheel_offset_z}"/>
    </joint>
    <link name="front_caster_wheel">
@@ -138,5 +231,5 @@
          <origin xyz="0.0 0.0 0.0"/>
          <geometry>
-            <sphere radius="0.041"/>
+            <sphere radius="${caster_wheel_radius}"/>
          </geometry>
          <material name="black"/>
@@ -145,33 +238,15 @@
          <origin xyz="0.0 0.0 0.0"/>
          <geometry>
-            <sphere radius="0.041"/>
-         </geometry>
-      </collision>
-      <xacro:inertial_sphere mass="0.15" radius="0.041">
+            <sphere radius="${caster_wheel_radius}"/>
+         </geometry>
+      </collision>
+      <xacro:inertial_sphere mass="${caster_wheel_mass}" radius="${caster_wheel_radius}">
          <origin xyz="0.0 0.0 0.0" rpy="0.0 0.0 0.0"/>
       </xacro:inertial_sphere>
    </link>
-   <joint name="back_caster_wheel_joint" type="fixed">
-      <parent link="back_caster_holder"/>
-      <child link="back_caster_wheel"/>
-      <origin xyz="-0.035 0.0 -0.025"/>
-   </joint>
-   <link name="back_caster_wheel">
-      <visual>
-         <origin xyz="0.0 0.0 0.0"/>
-         <geometry>
-            <sphere radius="0.041"/>
-         </geometry>
-         <material name="black"/>
-      </visual>
-      <collision>
-         <origin xyz="0.0 0.0 0.0"/>
-         <geometry>
-            <sphere radius="0.041"/>
-         </geometry>
-      </collision>
-      <xacro:inertial_sphere mass="0.1" radius="0.041">
-         <origin xyz="0.0 0.0 0.0" rpy="0.0 0.0 0.0"/>
-      </xacro:inertial_sphere>
-   </link>
+   <gazebo reference="front_caster_wheel">
+      <material>Gazebo/Black</material>
+      <mu1 value="0.001"/>
+      <mu2 value="0.001"/>
+   </gazebo>
 </robot>

Commit message: fixed ros2_control sim_mode

File: description/robot.urdf.xacro (robot description, xacro)
@@ -3,4 +3,5 @@
    <!-- args -->
    <xacro:arg name="use_ros2_control" default="true"/>
+   <xacro:arg name="sim_mode" default="false"/>
    <!-- initialize xacro properties -->
    <xacro:include filename="inertial_macros.xacro"/>

File: description/ros2_control.xacro (robot description, xacro)
@@ -1,56 +1,61 @@
 <?xml version="1.0" encoding="UTF-8"?>
 <robot xmlns:xacro="http://www.ros.org/wiki/xacro">
-   <ros2_control name="RealRobot" type="system">
-      <hardware>
-         <plugin>diffdrive_arduino/DiffDriveArduino</plugin>
-         <param name="left_wheel_name">left_wheel_joint</param>
-         <param name="right_wheel_name">right_wheel_joint</param>
-         <param name="loop_rate">30</param>
-         <param name="device">/dev/ttyACM0</param>
-         <param name="baud_rate">57600</param>
-         <param name="timeout">1000</param>
-         <param name="enc_counts_per_rev">2800</param>
-      </hardware>
-      <joint name="left_wheel_joint">
-         <command_interface name="velocity">
-            <param name="min">-10</param>
-            <param name="max">10</param>
-         </command_interface>
-         <state_interface name="velocity"/>
-         <state_interface name="position"/>
-      </joint>
-      <joint name="right_wheel_joint">
-         <command_interface name="velocity">
-            <param name="min">-10</param>
-            <param name="max">10</param>
-         </command_interface>
-         <state_interface name="velocity"/>
-         <state_interface name="position"/>
-      </joint>
-   </ros2_control>
-   <!-- <ros2_control name="GazeboSystem" type="system">
-      <hardware>
-         <plugin>gazebo_ros2_control/GazeboSystem</plugin>
-      </hardware>
-      <joint name="left_wheel_joint">
-         <command_interface name="velocity">
-            <param name="min">-10</param>
-            <param name="max">10</param>
-         </command_interface>
-         <state_interface name="velocity"/>
-         <state_interface name="position"/>
-      </joint>
-      <joint name="right_wheel_joint">
-         <command_interface name="velocity">
-            <param name="min">-10</param>
-            <param name="max">10</param>
-         </command_interface>
-         <state_interface name="velocity"/>
-         <state_interface name="position"/>
-      </joint>
-   </ros2_control> -->
+   <xacro:unless value="$(arg sim_mode)">
+      <ros2_control name="RealRobot" type="system">
+         <hardware>
+            <plugin>diffdrive_arduino/DiffDriveArduino</plugin>
+            <param name="left_wheel_name">left_wheel_joint</param>
+            <param name="right_wheel_name">right_wheel_joint</param>
+            <param name="loop_rate">30</param>
+            <param name="device">/dev/ttyACM0</param>
+            <param name="baud_rate">57600</param>
+            <param name="timeout">1000</param>
+            <param name="enc_counts_per_rev">2800</param>
+         </hardware>
+         <joint name="left_wheel_joint">
+            <command_interface name="velocity">
+               <param name="min">-10</param>
+               <param name="max">10</param>
+            </command_interface>
+            <state_interface name="velocity"/>
+            <state_interface name="position"/>
+         </joint>
+         <joint name="right_wheel_joint">
+            <command_interface name="velocity">
+               <param name="min">-10</param>
+               <param name="max">10</param>
+            </command_interface>
+            <state_interface name="velocity"/>
+            <state_interface name="position"/>
+         </joint>
+      </ros2_control>
+   </xacro:unless>
+   <xacro:if value="$(arg sim_mode)">
+      <ros2_control name="GazeboSystem" type="system">
+         <hardware>
+            <plugin>gazebo_ros2_control/GazeboSystem</plugin>
+         </hardware>
+         <joint name="left_wheel_joint">
+            <command_interface name="velocity">
+               <param name="min">-10</param>
+               <param name="max">10</param>
+            </command_interface>
+            <state_interface name="velocity"/>
+            <state_interface name="position"/>
+         </joint>
+         <joint name="right_wheel_joint">
+            <command_interface name="velocity">
+               <param name="min">-10</param>
+               <param name="max">10</param>
+            </command_interface>
+            <state_interface name="velocity"/>
+            <state_interface name="position"/>
+         </joint>
+      </ros2_control>
+   </xacro:if>
    <gazebo>
       <plugin name="gazebo_ros2_control" filename="libgazebo_ros2_control.so">
          <parameters>$(find robot_bringup)/config/controllers.yaml</parameters>
+         <parameters>$(find robot_bringup)/config/gazebo_controllers.yaml</parameters>
       </plugin>
    </gazebo>
