Commit message: added slam_toolbox

File: description/robot_core.xacro (robot description, xacro)
@@ -3,4 +3,11 @@
    <!-- BASE LINK -->
    <link name="base_link"></link>
+   <!-- BASE FOOTPRINT -->
+   <joint name="base_footprint_joint" type="fixed">
+      <parent link="base_link"/>
+      <child link="base_footprint"/>
+      <origin xyz="0 0 0" rpy="0 0 0"/>
+   </joint>
+   <link name="base_footprint"></link>
    <!-- CHASSIS -->
    <joint name="chassis_joint" type="fixed">
